Commit message: drones positioned properly

File: rotors_description/urdf/collaborative/four_hummingbirds_payload.xacro (robot description, xacro)
@@ -52,5 +52,5 @@
 		parent_link_holder = "${name_holder_0}"
 		sphere_joint_name = "sphere_${name_quad_0}_${name_holder_0}"
-		offset_holder = "${holder_height}+0.5"
+		offset_holder = "${holder_height+0.05}"
 		>
 	</xacro:hummingbird_with_payload_offset>

File: rotors_description/urdf/collaborative/multirotor_base.xacro (robot description, xacro)
@@ -32,8 +32,9 @@
   </xacro:macro>
   <!-- Macro for sphere joint with force sensor -->
-  <xacro:macro name="sphere_joint" params = "robot_namespace joint_velocity_limit joint_effort_limit parent_link_holder *origin_from_parent">
+  <xacro:macro name="sphere_joint" params = "robot_namespace joint_velocity_limit joint_effort_limit parent_link_holder offset_holder *origin_from_parent">
     <joint name="${robot_namespace}/sphjoint1" type="continuous">
       <parent link="${parent_link_holder}"/>
       <child link="${robot_namespace}/sphlink_z"/>
+      <origin xyz="0 0 ${offset_holder}" rpy="0 0 0"/>
       <axis xyz="0 0 1" />
       <insert_block name="origin_from_parent"/>
@@ -49,4 +50,5 @@
       <parent link="${robot_namespace}/sphlink_z"/>
       <child link="${robot_namespace}/sphlink_y"/>
+      <!-- <origin xyz="0 0 ${offset_holder}" rpy="0 0 0"/> -->
       <axis xyz="0 1 0" />
       <limit lower="${-pi/4}" upper="${pi/4}" velocity="${joint_velocity_limit}" effort="${joint_effort_limit}" />
@@ -61,4 +63,5 @@
       <parent link="${robot_namespace}/sphlink_y"/>
       <child link="${robot_namespace}/sphlink_x"/>
+      <!-- <origin xyz="0 0 ${offset_holder}" rpy="0 0 0"/> -->
       <axis xyz="1 0 0" />
       <limit lower="${-pi/4}" upper="${pi/4}" velocity="${joint_velocity_limit}" effort="${joint_effort_limit}" />
@@ -108,4 +111,5 @@
       joint_velocity_limit = "${joint_velocity_limit}"
       joint_effort_limit = "${joint_effort_limit}"
+      offset_holder = "${offset_holder}"
       >
       <origin xyz="0 0 ${offset_holder}" rpy="0 0 0"/>

Commit message: able to control the attitude of drones

File: rotors_description/urdf/collaborative/four_hummingbirds_payload.xacro (robot description, xacro)
@@ -33,5 +33,5 @@
 	  <xacro:property name="holder_width" value ="0.05" />
 	  <xacro:property name="holder_height" value="1.2" />
-	  <xacro:property name="mass_holder" value="1.0" />
+	  <xacro:property name="mass_holder" value="0.03" />
 	<xacro:include filename="$(find rotors_description)/urdf/collaborative/component_snippets.xacro" />
 	<xacro:include filename="$(find rotors_description)/urdf/collaborative/hummingbird_payload_offset.xacro"/>

Commit message: payload holder weight playground

File: rotors_description/urdf/collaborative/four_hummingbirds_payload.xacro (robot description, xacro)
@@ -33,5 +33,5 @@
 	  <xacro:property name="holder_width" value ="0.05" />
 	  <xacro:property name="holder_height" value="1.2" />
-	  <xacro:property name="mass_holder" value="0.03" />
+	  <xacro:property name="mass_holder" value="0.05" />
 	<xacro:include filename="$(find rotors_description)/urdf/collaborative/component_snippets.xacro" />
 	<xacro:include filename="$(find rotors_description)/urdf/collaborative/hummingbird_payload_offset.xacro"/>
